File: pcb/EEC-IV-Reader.kicad_pcb (KiCad board)
At the start: 2 copper layers, 53 x 68.7 mm, 33 parts, among them J1 ARDUINO_1, J2 ARDUINO_2, J3 RS_485_DEBUG, J4 ARDUINO_3, J5 ARDUINO_4, J6 DISPLAY, J7 OBD, J8 I2C_DEBUG, J9 Vin_disconnect, SW1 BTN_UP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

Commit message: Improve board
Parts:
- added G***: LOGO, Library:mondeo, F.Cu at (55.9, 91.4)
- renumbered J8 to I2C, J3 to Serial, J9 to Vin
Other:
- board text added: "EEC IV Reader"
- board text added: "OBD PWR"
- board text added: "v0.3"

Commit message: Update PCB
Parts:
- removed I2C: I2C_DEBUG, Connector_PinHeader_2.54mm:PinHeader_1x02_P2.54mm_Vertical
- removed Serial: RS_485_DEBUG, Connector_PinHeader_2.54mm:PinHeader_1x04_P2.54mm_Vertical
- removed Vin: Vin_disconnect, Connector_PinHeader_2.54mm:PinHeader_1x02_P2.54mm_Vertical
- added D2: D_Schottky, Diode_THT:D_A-405_P7.62mm_Horizontal, F.Cu at (80.0, 61.3)
- added D3: LED, LED_THT:LED_D3.0mm, F.Cu at (51.2, 73.4)
- added D4: LED, LED_THT:LED_D3.0mm, F.Cu at (51.2, 78.9)
- added J3: RS_485_DEBUG, Connector_PinHeader_2.54mm:PinHeader_1x04_P2.54mm_Vertical, F.Cu at (46.3, 37.5)
- added J8: I2C_DEBUG, Connector_PinHeader_2.54mm:PinHeader_1x02_P2.54mm_Vertical, F.Cu at (46.6, 76.9)
- added J9: Vin_disconnect, Connector_PinHeader_2.54mm:PinHeader_1x02_P2.54mm_Vertical, F.Cu at (87.7, 57.1)
- added R13: 160, Resistor_THT:R_Axial_DIN0207_L6.3mm_D2.5mm_P7.62mm_Horizontal, F.Cu at (68.4, 63.2)
- added R14: 160, Resistor_THT:R_Axial_DIN0207_L6.3mm_D2.5mm_P7.62mm_Horizontal, F.Cu at (68.3, 67.1)
- J1, J5: footprint Connector_PinHeader_2.54mm:PinHeader_1x08_P2.54mm_Vertical -> Connector_PinSocket_2.54mm:PinSocket_1x08_P2.54mm_Vertical; moved to B.Cu
- J2: footprint Connector_PinHeader_2.54mm:PinHeader_1x06_P2.54mm_Vertical -> Connector_PinSocket_2.54mm:PinSocket_1x06_P2.54mm_Vertical; moved to B.Cu
- J4: footprint Connector_PinHeader_2.54mm:PinHeader_1x10_P2.54mm_Vertical -> Connector_PinSocket_2.54mm:PinSocket_1x10_P2.54mm_Vertical; moved to B.Cu
- J6: footprint Connector_PinHeader_2.54mm:PinHeader_1x04_P2.54mm_Vertical -> Connector_PinSocket_2.54mm:PinSocket_1x04_P2.54mm_Vertical
- moved R1 1.48 mm to (60.7, 76.1)
- turned J1 to 0 degrees
- turned J2 to 0 degrees
- turned J4 to 0 degrees
- turned J5 to 0 degrees
Connections:
- J1 pad 1: Net-(J1-Pad1) -> unconnected-(J1-Pad1)
- J1 pad 2: Net-(J1-Pad2) -> unconnected-(J1-Pad2)
- J1 pad 3: Net-(J1-Pad3) -> unconnected-(J1-Pad3)
- J1 pad 4: Net-(J1-Pad4) -> unconnected-(J1-Pad4)
- J2 pad 1: Net-(J2-Pad1) -> unconnected-(J2-Pad1)
- J2 pad 2: Net-(J2-Pad2) -> unconnected-(J2-Pad2)
- J2 pad 3: Net-(J2-Pad3) -> unconnected-(J2-Pad3)
- J2 pad 4: Net-(J2-Pad4) -> unconnected-(J2-Pad4)
- J2 pad 5: Net-(J2-Pad5) -> unconnected-(J2-Pad5)
- J2 pad 6: Net-(J2-Pad6) -> unconnected-(J2-Pad6)
- J4 pad 3: Net-(J4-Pad3) -> unconnected-(J4-Pad3)
- J4 pad 5: Net-(J4-Pad5) -> unconnected-(J4-Pad5)
- J4 pad 6: Net-(J4-Pad6) -> unconnected-(J4-Pad6)
- J4 pad 7: Net-(J4-Pad7) -> unconnected-(J4-Pad7)
- J4 pad 8: Net-(J4-Pad8) -> unconnected-(J4-Pad8)
- J5 pad 2: Net-(J5-Pad2) -> unconnected-(J5-Pad2)
- J5 pad 3: Net-(J5-Pad3) -> unconnected-(J5-Pad3)
- J5 pad 7: Net-(J5-Pad7) -> unconnected-(J5-Pad7)
- J5 pad 8: Net-(J5-Pad8) -> unconnected-(J5-Pad8)
Routing:
- net 4: track 11.4 -> 44.4 mm
- net 2: track 26.0 -> 46.5 mm
- net Net-(D4-Pad2): track 0.00 -> 14.7 mm
- net Net-(D3-Pad2): track 0.00 -> 13.1 mm
- net +5V: track 139.1 -> 149.3 mm
- net /8V: track 16.2 -> 23.3 mm
- net Net-(D2-Pad2): track 0.00 -> 4.26 mm
- net VIN: track 4.84 -> 7.83 mm
- net 9: track 49.7 -> 52.7 mm
- net 8: track 61.8 -> 63.7 mm
Other:
- board text added: "12V D- D+ GND"
- board text added: "DI"
- board text added: "DOWN"
- board text added: "GND"
- board text added: "RO"
- board text added: "SCL SDA"
- board text added: "SELECT"
- board text added: "UP"
- board text added: "Vin Disc."
